File: breadboard-pwr.kicad_sch (KiCad schematic)
At the start: 11 parts, among them J1 Conn_02x03_Odd_Even, J2 Conn_02x03_Odd_Even, J3 Conn_02x04_Odd_Even, U1 LM337_TO220, U2 LM7805_TO220

Commit message: Add image and schematic
Parts:
- C1, C2: value (none) -> 10uF
- R1: value (none) -> 120
Changed lines of the file:
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@@
 (kicad_sch (version 20211123) (generator eeschema)
-  (paper "A4")
+  (paper "A5")
   (junction (at 55.88 69.85) (diameter 0) (color 0 0 0 0)
   )
@@
       (effects (font (size 1.27 1.27)) (justify right))
     )
-    (property "Value" "" (id 1) (at 107.95 38.646 0)
+    (property "Value" "10uF" (id 1) (at 107.95 38.646 0)
       (effects (font (size 1.27 1.27)) (justify right))
     )
@@
       (effects (font (size 1.27 1.27)) (justify left))
     )
-    (property "Value" "" (id 1) (at 140.97 39.916 0)
+    (property "Value" "10uF" (id 1) (at 140.97 39.916 0)
       (effects (font (size 1.27 1.27)) (justify left))
     )
@@
       (effects (font (size 1.27 1.27)) (justify left))
     )
-    (property "Value" "" (id 1) (at 132.08 39.3699 0)
-      (effects (font (size 1.27 1.27)) (justify left))
-    )
+    (property "Value" "120" (id 1) (at 132.08 39.3699 0)
+      (effects (font (size 1.27 1.27)) (justify left))
+    )
